Commit message: Update urdf to match old info yaml

File: xarmrob_util/src/urdf/robot-xarm.urdf (robot description, URDF)
Before this commit: robot visual, 8 links, 7 joints
Joints:
- joint base_joint: limit lower=-2.6 upper=2.6 effort=1000.0 velocity=.5 -> lower=-2.09 upper=2.09 effort=1000.0 velocity=.5
- joint fingers_joint: limit lower=-1.95 upper=1.95 effort=1000.0 velocity=.5 -> lower=-1.91 upper=1.91 effort=1000.0 velocity=.5
- joint forearm_joint: limit lower=-1.95 upper=1.95 effort=1000.0 velocity=.5 -> lower=-1.91 upper=1.91 effort=1000.0 velocity=.5
- joint gripper: limit lower=0 upper=1.58 effort=1000.0 velocity=.5 -> lower=0 upper=1.57 effort=1000.0 velocity=.5
- joint shoulder_joint: limit lower=-3.14 upper=0 effort=1000.0 velocity=.5 -> lower=-2.96 upper=-0.18 effort=1000.0 velocity=.5
- joint wrist_joint: limit lower=-1.75 upper=1.75 effort=1000.0 velocity=.5 -> lower=-1.57 upper=1.57 effort=1000.0 velocity=.5

Commit message: Restrict forearm joint to +/- 90 degrees

File: xarmrob_util/src/urdf/robot-xarm.urdf (robot description, URDF)
Before this commit: robot visual, 8 links, 7 joints
Joints:
- joint forearm_joint: limit lower=-1.91 upper=1.91 effort=1000.0 velocity=.5 -> lower=-1.57 upper=1.57 effort=1000.0 velocity=.5

Commit message: Restrict finger joint to +/- 90 degrees

File: xarmrob_util/src/urdf/robot-xarm.urdf (robot description, URDF)
Before this commit: robot visual, 8 links, 7 joints
Joints:
- joint fingers_joint: limit lower=-1.91 upper=1.91 effort=1000.0 velocity=.5 -> lower=-1.57 upper=1.57 effort=1000.0 velocity=.5
